File: MCU - Marv Communication Unit/Eagle/MCU_Power_PCB_Rev1/MCU_Power_PCB_Rev1/MCU_Power_PCB_Rev1.brd (EAGLE design)
At the start: 32 parts, among them IC1 LTC2955CTS8-1#TRMPBF, J1 39-30-3035, J2 39-30-3035, J3 39-30-3046, J4 3522-2, Q1 2N7002PW,115, Q2 2N7002PW,115, Q3 2N7002PW,115

Commit message: -
Parts:
- removed IC1: LTC2955CTS8-1#TRMPBF, LTC2955CTS8-1#TRMPBF:SOT65P280X100-8N
- added C1: 1 uF, CASE-RCL:C0603
- added C2: 0.1 uF, CASE-RCL:C0603
- added D11: 12.00V, diode:SOD-123_MINI-SMA
- added IC3: CD4011BM, CD4011BM:SOIC127P600X175-14N
- added J5: 3522-2, 3522-2:35222
- added J6, J7, J8, J9: 39-30-0020, 39-30-0020:39-30-1020_1
- added K1: V23079A1003B301, CASE-Relay:413937885
- added Q4: IPD90P03P4-04, IPD90P03P4-04:PG-TO252-3-11
- added Q5, Q6: 2N7002PW,115, CASE-Transistors:SOT323
- added R10, R11, R13: 100K, CASE-RCL:R0603
- added R12: (no value), CASE-RCL:R0603
- added R14: 10K, CASE-RCL:R0603
- D6: value 10.00V -> 10.10V
- Q1: value 2N7002PW,115 -> IPD90P03P4-04; device CASE-Transistors:SOT323 -> IPD90P03P4-04:PG-TO252-3-11
- R7: value 10K -> 100K
- R9: value 100K -> (none)
- moved Q2 159.9 mm to (-118.5, -232.0)
- moved Q3 159.9 mm to (-118.5, -238.5)
- moved R8 154.2 mm to (-118.5, -219.0)
- moved R7 148.8 mm to (-118.5, -207.0)
- moved Q1 147.1 mm to (-113.0, -194.5)
- moved R9 146.7 mm to (-118.5, -224.0)
Connections:
- removed net N$2: D1.A, R1.1
- new net A_OFF: IC3.3, IC3.5, IC3.6, R8.2, R9.2
- new net A_ON: IC3.4, R12.1, R7.2
- new net N$14: Q2.1, Q3.1, Q5.3, R13.2, R14.1
- new net N$18: J1.3, Q4.3
- new net N$19: D11.C, J5.2, J5.4, Q4.2
- new net N$20: D11.A, Q4.1, R10.1
- new net N$21: C1.1, J3.1, K1.4, Q2.3, Q3.2, R8.1
- new net N$23: J2.2, J4.1, J4.3
- new net VCC: D6.C, J6.2, J7.2, J8.2, J9.2, Q1.3, R14.2
- net +12V: now also IC3.14, J4.2, J4.4, J5.1, J5.3, Q1.2; no longer D6.C, R1.2, R7.1
- net GND: now also C1.2, C2.2, D1.K, IC3.7, J1.1, J2.1, J6.1, J7.1, J8.1, J9.1, K1.12, Q5.2, Q6.2, R10.2, R11.2, R13.1, R6.1; no longer IC1.4, Q1.2, Q2.2, R6.2, R8.2, R9.2
- net N$1: now also K1.1, Q5.1, R6.2; no longer Q1.1, R6.1
- net N$11: now also Q1.1, R12.2, R9.1; no longer Q1.3, Q2.1, R7.2, R8.1
- net N$12: now also D1.A, Q6.3, R1.2; no longer D1.K, Q3.3
- net N$15: now also C2.1, IC3.1, IC3.2, J3.2, K1.3, Q2.2, Q3.3, R7.1; no longer Q2.3, Q3.2
- net N$16: now also R1.1; no longer Q3.1, R9.1
- net N$4: now also Q6.1, R11.1

Commit message: finished board
Parts:
- removed C1: 1 uF, CASE-RCL:C0603
- removed C2: 0.1 uF, CASE-RCL:C0603
- removed IC3: CD4011BM, CD4011BM:SOIC127P600X175-14N
- removed K1: V23079A1003B301, CASE-Relay:413937885
- removed Q2, Q3, Q5: 2N7002PW,115, CASE-Transistors:SOT323
- removed R13, R6, R7, R8: 100K, CASE-RCL:R0603
- removed R14: 10K, CASE-RCL:R0603
- added C3, C6: 0.1 uF, CASE-RCL:C0603
- added C4, C5: 0.033 uF, CASE-RCL:C0603
- added D12, D14: 2.5V, diode:SOD-123_MINI-SMA
- added D13: 3.3V, diode:SOD-123_MINI-SMA
- added IC1: LTC2950ITS8-2#TRMPBF, LTC2950ITS8-2#TRMPBF:SOT65P280X100-8N
- D10: value 12.12V -> 10.0V
- D6: value 10.10V -> 1.8V
- D7: value 10.00V -> 6.0V
- D8: value 10.71V -> 6.0V
- D9: value 11.38V -> 6.0V
- R12: value (none) -> 33K
- R9: value (none) -> 510K
- moved R12 261.8 mm to (-25.0, 17.0), flipped to the bottom, turned to 270 degrees
- moved R9 257.4 mm to (-28.0, 17.0), flipped to the bottom, turned to 90 degrees
- moved R11 245.2 mm to (29.0, 13.5), flipped to the bottom, turned to 270 degrees
- moved Q6 238.5 mm to (26.0, 13.5), flipped to the bottom, turned to 270 degrees
- moved Q1 223.5 mm to (-24.0, 10.5), flipped to the bottom
- moved D11 204.3 mm to (-6.00, 5.00), flipped to the bottom, turned to 90 degrees
- moved R10 196.8 mm to (-3.00, 0.00), flipped to the bottom, turned to 270 degrees
- moved J9 187.5 mm to (-50.0, 12.0), flipped to the bottom, turned to 90 degrees
- moved Q4 181.8 mm to (-18.0, 5.00), flipped to the bottom, turned to 270 degrees
- moved J6 176.5 mm to (-50.0, 4.00), flipped to the bottom, turned to 90 degrees
- moved J5 171.4 mm to (10.5, -1.50), flipped to the bottom
- moved J7 169.1 mm to (-50.0, -4.00), flipped to the bottom, turned to 90 degrees
- moved J8 162.1 mm to (-50.0, -12.0), flipped to the bottom, turned to 90 degrees
- moved J4 151.2 mm to (-16.5, -6.00), flipped to the bottom, turned to 180 degrees
- moved J3 134.1 mm to (14.0, -10.5), flipped to the bottom
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Connections:
- removed net A_OFF: IC3.3, IC3.5, IC3.6, R8.2, R9.2
- removed net A_ON: IC3.4, R12.1, R7.2
- removed net N$14 (its old number): Q2.1, Q3.1, Q5.3, R13.2, R14.1
- new net N$17: C5.1, IC1.7
- new net N$2: C4.1, IC1.3
- new net N$22: D14.A, Q6.1, R11.1
- new net N$24: C6.1, IC1.5, IC1.8, R12.1, R9.2
- new net N$25: IC1.6, Q1.1
- net +12V: now also C3.1, D11.C, IC1.1, Q4.2; no longer IC3.14, J5.1, J5.3
- net GND: now also C3.2, C4.2, C5.2, C6.2, IC1.4, J3.2, J3.4, R12.2; no longer C1.2, C2.2, IC3.7, K1.12, Q5.2, R13.1, R6.1
- net N$1: now also J5.1, J5.3, Q4.3; no longer D6.A, K1.1, Q5.1, R6.2
- net N$11: now also IC1.2, J3.3; no longer Q1.1, R12.2, R9.1
- net N$15: now also D6.A, D7.C; no longer C2.1, IC3.1, IC3.2, J3.2, K1.3, Q2.2, Q3.3, R7.1
- net N$16: now also D12.C, D13.C, D6.C; no longer D7.C, D8.C, D9.C
- net N$18: now also J5.2, J5.4; no longer Q4.3
- net N$19: now also D12.A, D8.C; no longer D11.C, J5.2, J5.4, Q4.2
- net N$21: now also D13.A, D9.C; no longer C1.1, J3.1, K1.4, Q2.3, Q3.2, R8.1
- net N$4: now also D14.C; no longer Q6.1, R11.1
- net VCC: now also J3.1, R9.1; no longer D6.C, R14.2
Routing:
- net +12V: track 0.00 -> 89.1 mm, vias 0 -> 2
- net N$11: track 0.00 -> 64.2 mm, vias 0 -> 1
- net N$16: track 0.00 -> 63.5 mm
- net VCC: track 0.00 -> 53.8 mm
- net N$13: track 0.00 -> 26.4 mm
- net N$25: track 0.00 -> 22.1 mm, vias 0 -> 2
- net N$22: track 0.00 -> 14.2 mm
- net N$24: track 0.00 -> 12.1 mm
- net N$4: track 0.00 -> 11.3 mm
- net N$20: track 0.00 -> 11.2 mm
- net N$12: track 0.00 -> 6.19 mm
- net N$2: track 0.00 -> 5.25 mm
- net N$17: track 0.00 -> 4.69 mm
- net N$9: track 0.00 -> 3.76 mm
- net N$8: track 0.00 -> 3.76 mm
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- added copper zone on layer 16, net +12V
- added copper zone on layer 1, net GND
- added copper zone on layer 16, net GND
- added copper zone on layer 1, net N$1
- added copper zone on layer 16, net N$14
- added copper zone on layer 16, net N$18
- added copper zone on layer 16, net VCC
Other:
- board outline added: 100 x 50 mm
- board text added: "12V"
- board text added: "ATO 7.5A"
- board text added: "Battery port"
- board text added: "Charging port"
- board text added: "GND"
- board text added: "LED+"
- board text added: "LED-"
- board text added: "MARV - MCU Power PCB Rev1, 21.11.05"
- board text added: "PB"
- board text added: "PWR_OUT"
- board text added: "Pushbutton"
