File: MCU - Marv Communication Unit/Eagle/MCU_Power_PCB_Rev1/MCU_Power_PCB_Rev1/MCU_Power_PCB_Rev1.sch (EAGLE design)
At the start: 49 parts, among them IC3 CD4011BM, J1 39-30-3035, J2 39-30-3035, J3 39-30-3046, J4 3522-2, J5 3522-2, J6 39-30-0020, J7 39-30-0020, J8 39-30-0020, J9 39-30-0020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

Commit message: finished board
Parts:
- removed C1: 1 uF, CASE-RCL:C0603
- removed C2: 0.1 uF, CASE-RCL:C0603
- removed IC3: CD4011BM, CD4011BM:CD4011BM
- removed K1: V23079A1003B301, CASE-Relay:V23079A1003B301
- removed Q2, Q3, Q5: 2N7002PW,115, CASE-Transistors:2N7002PW,115
- removed R13, R6, R7, R8: 100K, CASE-RCL:R0603
- removed R14: 10K, CASE-RCL:R0603
- added C3, C6: 0.1 uF, CASE-RCL:C0603
- added C4, C5: 0.033 uF, CASE-RCL:C0603
- added D12, D14: 2.5V, diode:CGRM4001-G
- added D13: 3.3V, diode:CGRM4001-G
- added IC1: LTC2950ITS8-2#TRMPBF, LTC2950ITS8-2#TRMPBF:LTC2950ITS8-2#TRMPBF
- D10: value 12.12V -> 10.0V
- D6: value 10.10V -> 1.8V
- D7: value 10.00V -> 6.0V
- D8: value 10.71V -> 6.0V
- D9: value 11.38V -> 6.0V
- R12: value (none) -> 33K
- R9: value (none) -> 510K
Connections:
- removed net A_OFF: IC3.C, IC3.D, IC3.J=!AB, R8.2, R9.2
- removed net A_ON: IC3.K=!CD, R12.1, R7.2
- removed net N$14 (its old number): Q2.G, Q3.G, Q5.D, R13.2, R14.1
- new net N$17: C5.1, IC1.OFFT
- new net N$2: C4.1, IC1.ONT
- new net N$22: D14.A, Q6.G, R11.1
- new net N$24: C6.1, IC1.!INT, IC1.!KILL, R12.1, R9.2
- new net N$25: IC1.EN/!EN, Q1.G
- net +12V: now also C3.1, D11.C, IC1.VIN, Q4.S; no longer IC3.VDD, J5.1, J5.3
- net GND: now also C3.2, C4.2, C5.2, C6.2, IC1.GND, J3.2, J3.4, R12.2; no longer C1.2, C2.2, IC3.VSS, K1.-, Q5.S, R13.1, R6.1
- net N$1: now also J5.1, J5.3, Q4.D; no longer D6.A, K1.+, Q5.G, R6.2
- net N$11: now also IC1.!PB, J3.3; no longer Q1.G, R12.2, R9.1
- net N$15: now also D6.A, D7.C; no longer C2.1, IC3.A, IC3.B, J3.2, K1.NC_1, Q2.S, Q3.D, R7.1
- net N$16: now also D12.C, D13.C, D6.C; no longer D7.C, D8.C, D9.C
- net N$18: now also J5.2, J5.4; no longer Q4.D
- net N$19: now also D12.A, D8.C; no longer D11.C, J5.2, J5.4, Q4.S
- net N$21: now also D13.A, D9.C; no longer C1.1, J3.1, K1.COM_1, Q2.D, Q3.S, R8.1
- net N$4: now also D14.C; no longer Q6.G, R11.1
- net VCC: now also J3.1, R9.1; no longer D6.C, R14.2
Other:
- note added: "1. GND 2. 12V 3. NC"
- note added: "1. GND 2. NC 3. 12V"
- note added: "1. GND 2. VCC"
- note added: "1. LED+ 2. LED- 3. PB+ 4. PB-"
- note added: "Battery port fuse - 7.5A"
- note added: "Battery status LEDs"
- note added: "CHALMERS"
- note added: "Mounting holes"
- note added: "Power input/output, fuses"
- note added: "Pushbutton controller/voltage monitor"
- note added: "Should cut power at ~9.9V IC cuts power under 0.6V !KILL"
- note added: "Viktor Lindström"
- note added: "~10.0V"
- note added: "~10.7V"
- note added: "~11.6V"
- note added: "~12.2V"
- note removed: "Power out fuse - 7.5A"
- moved on the sheet: D1, D10, D11, D2, D3, D4, D5, D6, D7, D8, D9, J1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
